Commit message: Gazebo backend implementation

File: src/portamail_navigator/urdf/portamail.urdf (robot description, URDF)
Before this commit: robot portamail_navigator, 5 links, 4 joints
Links:
- added link laser, mass 0.125; collision cylinder length=0.05 radius=0.04; visual cylinder length=0.05 radius=0.04
Joints:
- added joint laser_joint: type fixed, parent base_link, child laser, origin xyz=0.1 0.0 0.15 rpy=0 0 0

Commit message: Revert "Gazebo backend implementation"
This reverts commit eee85aba5fe585419b00bd43f07e732239cb2eea.

File: src/portamail_navigator/urdf/portamail.urdf (robot description, URDF)
Before this commit: robot portamail_navigator, 6 links, 5 joints
Links:
- removed link laser
Joints:
- removed joint laser_joint

Commit message: Claude code 🎉
First look at the use of claude code. It's been loaded with what I hope if the most up to date and accurate understanding of the software, electrical, and mechanical framework of this project.

File: src/portamail_navigator/urdf/portamail.urdf (robot description, URDF)
Before this commit: robot portamail_navigator, 5 links, 4 joints
Links:
- added link imu_link
- added link laser
- added link ultrasonic_link
Joints:
- added joint imu_joint: type fixed, parent base_link, child imu_link, origin xyz=0.0 0.0 0.05 rpy=0 0 0
- added joint laser_joint: type fixed, parent base_link, child laser, origin xyz=0.1 0.0 0.3 rpy=0 0 0
- added joint ultrasonic_joint: type fixed, parent base_link, child ultrasonic_link, origin xyz=0.2 0.0 0.05 rpy=0 0 0
